File: hardware/funbox_v3_midi_exp/Midi.kicad_sch (KiCad schematic)
At the start: 7 parts, among them U3 TL072, U5 H11L1

Commit message: Updated to version 3.1, fix expression, adjusted pieces
Parts:
- removed U3: TL072, Package_DIP:DIP-8_W7.62mm, symbol Amplifier_Operational:TL072
- added U3: MCP6002, Package_DIP:DIP-8_W7.62mm, symbol Amplifier_Operational:MCP6002-xP
Connections:
- net 3V3_A: now also U3.3 (+)
- net 5V: now also U3.8 (V+)
- net EXPRESSION_IN: now also U3.6 (-), U3.7
- net EXPRESSION_IN_JACK: now also U3.5 (+)
- net EXPRESSION_REF: now also U3.1, U3.2 (-)
- net GND: now also U3.4 (V-)
